Commit message: rename package name and file path for abb 150 320

File: abb_fabtory/urdf/abb_fabtory.urdf (robot description, URDF)
Before this commit: robot abb_fabtory, 15 links, 14 joints
Links:
- link base_link: geometry collision mesh filename=package://abb_irb6700_150_320/meshes/irb6700/collision/base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; visual mesh filename=package://abb_irb6700_150_320/meshes/irb6700/visual/base_li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
- link cylinder: geometry collision mesh filename=package://abb_irb6700_150_320/meshes/irb6700/collision/cyli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; visual mesh filename=package://abb_irb6700_150_320/meshes/irb6700/visual/cylinde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
- link link_1: geometry collision mesh filename=package://abb_irb6700_150_320/meshes/irb6700/collision/link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; visual mesh filename=package://abb_irb6700_150_320/meshes/irb6700/visual/link_1.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
- link link_2: geometry collision mesh filename=package://abb_irb6700_150_320/meshes/irb6700_150_320/collis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; visual mesh filename=package://abb_irb6700_150_320/meshes/irb6700_150_320/visual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
- link link_3: geometry collision mesh filename=package://abb_irb6700_150_320/meshes/irb6700_150_320/collis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; visual mesh filename=package://abb_irb6700_150_320/meshes/irb6700_150_320/visual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
- link link_4: geometry collision mesh filename=package://abb_irb6700_150_320/meshes/irb6700_150_320/collis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; visual mesh filename=package://abb_irb6700_150_320/meshes/irb6700_150_320/visual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
- link link_5: geometry collision mesh filename=package://abb_irb6700_150_320/meshes/irb6700/collision/link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; visual mesh filename=package://abb_irb6700_150_320/meshes/irb6700/visual/link_5.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
- link link_6: geometry collision mesh filename=package://abb_irb6700_150_320/meshes/irb6700/collision/link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; visual mesh filename=package://abb_irb6700_150_320/meshes/irb6700/visual/link_6.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
- link piston: geometry collision mesh filename=package://abb_irb6700_150_320/meshes/irb6700/collision/pist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; visual mesh filename=package://abb_irb6700_150_320/meshes/irb6700/visual/piston.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

File: abb_irb6700_150_320/urdf/irb6700_150_320.urdf (robot description, URDF)
Before this commit: robot abb_irb6700_150_320, 12 links, 11 joints
Links:
- link base_link: geometry collision mesh filename=package://abb_irb6700_150_320/meshes/irb6700/collision/base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; visual mesh filename=package://abb_irb6700_150_320/meshes/irb6700/visual/base_li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
- link cylinder: geometry collision mesh filename=package://abb_irb6700_150_320/meshes/irb6700/collision/cyli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; visual mesh filename=package://abb_irb6700_150_320/meshes/irb6700/visual/cylinde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
- link link_1: geometry collision mesh filename=package://abb_irb6700_150_320/meshes/irb6700/collision/link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; visual mesh filename=package://abb_irb6700_150_320/meshes/irb6700/visual/link_1.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
- link link_2: geometry collision mesh filename=package://abb_irb6700_150_320/meshes/irb6700_150_320/collis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; visual mesh filename=package://abb_irb6700_150_320/meshes/irb6700_150_320/visual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
- link link_3: geometry collision mesh filename=package://abb_irb6700_150_320/meshes/irb6700_150_320/collis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; visual mesh filename=package://abb_irb6700_150_320/meshes/irb6700_150_320/visual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
- link link_4: geometry collision mesh filename=package://abb_irb6700_150_320/meshes/irb6700_150_320/collis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; visual mesh filename=package://abb_irb6700_150_320/meshes/irb6700_150_320/visual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
- link link_5: geometry collision mesh filename=package://abb_irb6700_150_320/meshes/irb6700/collision/link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; visual mesh filename=package://abb_irb6700_150_320/meshes/irb6700/visual/link_5.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
- link link_6: geometry collision mesh filename=package://abb_irb6700_150_320/meshes/irb6700/collision/link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; visual mesh filename=package://abb_irb6700_150_320/meshes/irb6700/visual/link_6.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
- link piston: geometry collision mesh filename=package://abb_irb6700_150_320/meshes/irb6700/collision/pist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; visual mesh filename=package://abb_irb6700_150_320/meshes/irb6700/visual/piston.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

File: abb_irb6700_150_320/urdf/irb6700_150_320_macro.xacro (robot description, xacro)
@@ -1,5 +1,5 @@
 <?xml version="1.0"?>
 <robot xmlns:xacro="http://ros.org/wiki/xacro">
-  <xacro:macro name="abb_irb6700_235_265" params="prefix">
+  <xacro:macro name="abb_irb6700_150_320" params="prefix">
     <xacro:include filename="$(find abb_resources)/urdf/common_materials.xacro"/>
     <!-- link list -->
@@ -8,12 +8,12 @@
         <origin xyz="0 0 0" rpy="0 0 0" />
         <geometry>
-          <mesh filename="package://abb_irb6700_support/meshes/irb6700/visual/base_link.stl" />
-        </geometry>
-        <xacro:material_abb_white/>
-      </visual>
-      <collision>
-        <origin xyz="0 0 0" rpy="0 0 0" />
-        <geometry>
-          <mesh filename="package://abb_irb6700_support/meshes/irb6700/collision/base_link.stl" />
+          <mesh filename="package://abb_irb6700_150_320/meshes/irb6700/visual/base_link.stl" />
+        </geometry>
+        <xacro:material_abb_white/>
+      </visual>
+      <collision>
+        <origin xyz="0 0 0" rpy="0 0 0" />
+        <geometry>
+          <mesh filename="package://abb_irb6700_150_320/meshes/irb6700/collision/base_link.stl" />
         </geometry>
         <xacro:material_abb_yellow/>
@@ -24,12 +24,12 @@
         <origin xyz="0 0 0" rpy="0 0 0" />
         <geometry>
-          <mesh filename="package://abb_irb6700_support/meshes/irb6700/visual/link_1.stl" />
-        </geometry>
-        <xacro:material_abb_white/>
-      </visual>
-      <collision>
-        <origin xyz="0 0 0" rpy="0 0 0" />
-        <geometry>
-          <mesh filename="package://abb_irb6700_support/meshes/irb6700/collision/link_1.stl" />
+          <mesh filename="package://abb_irb6700_150_320/meshes/irb6700/visual/link_1.stl" />
+        </geometry>
+        <xacro:material_abb_white/>
+      </visual>
+      <collision>
+        <origin xyz="0 0 0" rpy="0 0 0" />
+        <geometry>
+          <mesh filename="package://abb_irb6700_150_320/meshes/irb6700/collision/link_1.stl" />
         </geometry>
         <xacro:material_abb_yellow/>
@@ -40,12 +40,12 @@
         <origin xyz="0 0 0" rpy="0 0 0" />
         <geometry>
-          <mesh filename="package://abb_irb6700_support/meshes/irb6700/visual/cylinder.stl" />
-        </geometry>
-        <xacro:material_abb_white/>
-      </visual>
-      <collision>
-        <origin xyz="0 0 0" rpy="0 0 0" />
-        <geometry>
-          <mesh filename="package://abb_irb6700_support/meshes/irb6700/collision/cylinder.stl" />
+          <mesh filename="package://abb_irb6700_150_320/meshes/irb6700/visual/cylinder.stl" />
+        </geometry>
+        <xacro:material_abb_white/>
+      </visual>
+      <collision>
+        <origin xyz="0 0 0" rpy="0 0 0" />
+        <geometry>
+          <mesh filename="package://abb_irb6700_150_320/meshes/irb6700/collision/cylinder.stl" />
         </geometry>
         <xacro:material_abb_yellow/>
@@ -56,12 +56,12 @@
         <origin xyz="0 0 0" rpy="0 0 0" />
         <geometry>
-          <mesh filename="package://abb_irb6700_support/meshes/irb6700/visual/piston.stl" />
-        </geometry>
-        <xacro:material_abb_white/>
-      </visual>
-      <collision>
-        <origin xyz="0 0 0" rpy="0 0 0" />
-        <geometry>
-          <mesh filename="package://abb_irb6700_support/meshes/irb6700/collision/piston.stl" />
+          <mesh filename="package://abb_irb6700_150_320/meshes/irb6700/visual/piston.stl" />
+        </geometry>
+        <xacro:material_abb_white/>
+      </visual>
+      <collision>
+        <origin xyz="0 0 0" rpy="0 0 0" />
+        <geometry>
+          <mesh filename="package://abb_irb6700_150_320/meshes/irb6700/collision/piston.stl" />
         </geometry>
         <xacro:material_abb_yellow/>
@@ -72,12 +72,12 @@
         <origin xyz="0 0 0" rpy="0 0 0" />
         <geometry>
-          <mesh filename="package://abb_irb6700_support/meshes/irb6700_235_265/visual/link_2.stl" />
-        </geometry>
-        <xacro:material_abb_white/>
-      </visual>
-      <collision>
-        <origin xyz="0 0 0" rpy="0 0 0" />
-        <geometry>
-          <mesh filename="package://abb_irb6700_support/meshes/irb6700_235_265/collision/link_2.stl" />
+          <mesh filename="package://abb_irb6700_150_320/meshes/irb6700_150_320/visual/link_2.stl" />
+        </geometry>
+        <xacro:material_abb_white/>
+      </visual>
+      <collision>
+        <origin xyz="0 0 0" rpy="0 0 0" />
+        <geometry>
+          <mesh filename="package://abb_irb6700_150_320/meshes/irb6700_150_320/collision/link_2.stl" />
         </geometry>
         <xacro:material_abb_yellow/>
@@ -88,12 +88,12 @@
         <origin xyz="0 0 0" rpy="0 0 0" />
         <geometry>
-          <mesh filename="package://abb_irb6700_support/meshes/irb6700_235_265/visual/link_3.stl" />
-        </geometry>
-        <xacro:material_abb_white/>
-      </visual>
-      <collision>
-        <origin xyz="0 0 0" rpy="0 0 0" />
-        <geometry>
-          <mesh filename="package://abb_irb6700_support/meshes/irb6700_235_265/collision/link_3.stl" />
+          <mesh filename="package://abb_irb6700_150_320/meshes/irb6700_150_320/visual/link_3.stl" />
+        </geometry>
+        <xacro:material_abb_white/>
+      </visual>
+      <collision>
+        <origin xyz="0 0 0" rpy="0 0 0" />
+        <geometry>
+          <mesh filename="package://abb_irb6700_150_320/meshes/irb6700_150_320/collision/link_3.stl" />
         </geometry>
         <xacro:material_abb_yellow/>
@@ -104,12 +104,12 @@
         <origin xyz="0 0 0" rpy="0 0 0" />
         <geometry>
-          <mesh filename="package://abb_irb6700_support/meshes/irb6700_235_265/visual/link_4.stl" />
-        </geometry>
-        <xacro:material_abb_white/>
-      </visual>
-      <collision>
-        <origin xyz="0 0 0" rpy="0 0 0" />
-        <geometry>
-          <mesh filename="package://abb_irb6700_support/meshes/irb6700_235_265/collision/link_4.stl" />
+          <mesh filename="package://abb_irb6700_150_320/meshes/irb6700_150_320/visual/link_4.stl" />
+        </geometry>
+        <xacro:material_abb_white/>
+      </visual>
+      <collision>
+        <origin xyz="0 0 0" rpy="0 0 0" />
+        <geometry>
+          <mesh filename="package://abb_irb6700_150_320/meshes/irb6700_150_320/collision/link_4.stl" />
         </geometry>
         <xacro:material_abb_yellow/>
@@ -120,12 +120,12 @@
         <origin xyz="0 0 0" rpy="0 0 0" />
         <geometry>
-          <mesh filename="package://abb_irb6700_support/meshes/irb6700/visual/link_5.stl" />
-        </geometry>
-        <xacro:material_abb_white/>
-      </visual>
-      <collision>
-        <origin xyz="0 0 0" rpy="0 0 0" />
-        <geometry>
-          <mesh filename="package://abb_irb6700_support/meshes/irb6700/collision/link_5.stl" />
+          <mesh filename="package://abb_irb6700_150_320/meshes/irb6700/visual/link_5.stl" />
+        </geometry>
+        <xacro:material_abb_white/>
+      </visual>
+      <collision>
+        <origin xyz="0 0 0" rpy="0 0 0" />
+        <geometry>
+          <mesh filename="package://abb_irb6700_150_320/meshes/irb6700/collision/link_5.stl" />
         </geometry>
         <xacro:material_abb_yellow/>
@@ -136,12 +136,12 @@
         <origin xyz="0 0 0" rpy="0 0 0" />
         <geometry>
-          <mesh filename="package://abb_irb6700_support/meshes/irb6700/visual/link_6.stl" />
-        </geometry>
-        <xacro:material_abb_white/>
-      </visual>
-      <collision>
-        <origin xyz="0 0 0" rpy="0 0 0" />
-        <geometry>
-          <mesh filename="package://abb_irb6700_support/meshes/irb6700/collision/link_6.stl" />
+          <mesh filename="package://abb_irb6700_150_320/meshes/irb6700/visual/link_6.stl" />
+        </geometry>
+        <xacro:material_abb_white/>
+      </visual>
+      <collision>
+        <origin xyz="0 0 0" rpy="0 0 0" />
+        <geometry>
+          <mesh filename="package://abb_irb6700_150_320/meshes/irb6700/collision/link_6.stl" />
         </geometry>
         <xacro:material_abb_yellow/>
@@ -153,5 +153,5 @@
       <child link="${prefix}link_1" />
       <axis xyz="0 0 1" />
-      <limit lower="-${radians(170)}" upper="${radians(170)}" effort="0" velocity="${radians(100)}" />
+      <limit lower="-${radians(170)}" upper="${radians(170)}" effort="0" velocity="${radians(110)}" />
     </joint>
     <joint name="${prefix}joint_2" type="revolute">
@@ -160,12 +160,12 @@
       <child link="${prefix}link_2" />
       <axis xyz="0 1 0" />
-      <limit lower="-${radians(65)}" upper="${radians(85)}" effort="0" velocity="${radians(90)}" />
+      <limit lower="-${radians(65)}" upper="${radians(85)}" effort="0" velocity="${radians(110)}" />
     </joint>
     <joint name="${prefix}joint_3" type="revolute">
-      <origin xyz="0 0 1.135" rpy="0 0 0" />
+      <origin xyz="0 0 1.280" rpy="0 0 0" />
       <parent link="${prefix}link_2" />
       <child link="${prefix}link_3" />
       <axis xyz="0 1 0" />
-      <limit lower="-${radians(180)}" upper="${radians(70)}" effort="0" velocity="${radians(90)}" />
+      <limit lower="-${radians(180)}" upper="${radians(70)}" effort="0" velocity="${radians(110)}" />
     </joint>
     <joint name="${prefix}joint_4" type="revolute">
@@ -174,12 +174,12 @@
       <child link="${prefix}link_4" />
       <axis xyz="1 0 0" />
-      <limit lower="-${radians(300)}" upper="${radians(300)}" effort="0" velocity="${radians(170)}" />
+      <limit lower="-${radians(300)}" upper="${radians(300)}" effort="0" velocity="${radians(190)}" />
     </joint>
     <joint name="${prefix}joint_5" type="revolute">
-      <origin xyz="1.1825 0 0" rpy="0 0 0" />
+      <origin xyz="1.593 0 0" rpy="0 0 0" />
       <parent link="${prefix}link_4" />
       <child link="${prefix}link_5" />
       <axis xyz="0 1 0" />
-      <limit lower="-${radians(130)}" upper="${radians(130)}" effort="0" velocity="${radians(120)}" />
+      <limit lower="-${radians(130)}" upper="${radians(130)}" effort="0" velocity="${radians(150)}" />
     </joint>
     <joint name="${prefix}joint_6" type="revolute">
@@ -188,5 +188,5 @@
       <child link="${prefix}link_6" />
       <axis xyz="1 0 0" />
-      <limit lower="-${radians(360)}" upper="${radians(360)}" effort="0" velocity="${radians(190)}" />
+      <limit lower="-${radians(360)}" upper="${radians(360)}" effort="0" velocity="${radians(210)}" />
     </joint>
     <joint name="${prefix}cylinder_joint" type="revolute">
