Commit message: urdf_updates

File: rbvogui_xl_ur10e_liftkit/urdf/rbvogui_xl_lift_ur10e.urdf (robot description, URDF)
Before this commit: robot rbvogui, 39 links, 38 joints
Joints:
- joint robot_ewellix_lift_base_joint: origin xyz=0.275 0.0 0.01 rpy=0 0 0 -> xyz=0.207 0.0 0.3 rpy=0 0 0

File: rbvogui_xl_ur10e_liftkit/urdf/rbvogui_xl_lift_ur10e_indoor.urdf (robot description, URDF)
Before this commit: robot rbvogui, 39 links, 38 joints
Joints:
- joint robot_ewellix_lift_base_joint: origin xyz=0.275 0.0 0.01 rpy=0 0 0 -> xyz=0.207 0.0 0.3 rpy=0 0 0

Commit message: urdf_changes

File: rbvogui_xl_ur10e_liftkit/urdf/rbvogui_xl_lift_ur10e.urdf (robot description, URDF)
Before this commit: robot rbvogui, 39 links, 38 joints
Joints:
- joint robot_ewellix_lift_base_joint: origin xyz=0.207 0.0 0.3 rpy=0 0 0 -> xyz=0.275 0.0 0.01 rpy=0 0 0

File: rbvogui_xl_ur10e_liftkit/urdf/rbvogui_xl_lift_ur10e_indoor.urdf (robot description, URDF)
Before this commit: robot rbvogui, 39 links, 38 joints
Joints:
- joint robot_ewellix_lift_base_joint: origin xyz=0.207 0.0 0.3 rpy=0 0 0 -> xyz=0.275 0.0 0.01 rpy=0 0 0
