Commit message: no more dae in urdf description of ur20

File: rbvogui_xl_ur20_liftkit/urdf/rbvogui_xl_ur20.urdf (robot description, URDF)
Before this commit: robot rbvogui, 39 links, 38 joints
Links:
- link robot_arm_base_link_inertia: geometry collision mesh filename=package://ur_description/meshes/ur20/collision/base.stl; visual mesh filename=package://ur_description/meshes/ur20/collision/base.stl
- link robot_arm_forearm_link: geometry collision mesh filename=package://ur_description/meshes/ur20/collision/forearm.stl; visual mesh filename=package://ur_description/meshes/ur20/collision/forearm.stl
- link robot_arm_shoulder_link: geometry collision mesh filename=package://ur_description/meshes/ur20/collision/shoulder.stl; visual mesh filename=package://ur_description/meshes/ur20/collision/shoulder.stl
- link robot_arm_upper_arm_link: geometry collision mesh filename=package://ur_description/meshes/ur20/collision/upperarm.stl; visual mesh filename=package://ur_description/meshes/ur20/collision/upperarm.stl
- link robot_arm_wrist_1_link: geometry collision mesh filename=package://ur_description/meshes/ur20/collision/wrist1.stl; visual mesh filename=package://ur_description/meshes/ur20/collision/wrist1.stl
- link robot_arm_wrist_2_link: geometry collision mesh filename=package://ur_description/meshes/ur20/collision/wrist2.stl; visual mesh filename=package://ur_description/meshes/ur20/collision/wrist2.stl
- link robot_arm_wrist_3_link: geometry collision mesh filename=package://ur_description/meshes/ur20/collision/wrist3.stl; visual mesh filename=package://ur_description/meshes/ur20/collision/wrist3.stl
- link robot_front_rgbd_camera_link: geometry collision mesh filename=package://robotnik_sensors/meshes/orbbec_astra.dae; visual mesh filename=package://robotnik_sensors/meshes/orbbec_astra.stl
